File: boards/PoE_Stepper_Driver/PoE_Stepper_Driver.kicad_pcb (KiCad board)
At the start: 2 copper layers, 99.1 x 71.1 mm, 123 parts, among them J1 RJ45, J2 Motor, J3 Limits, Q1 NMOS_POE, Q10 NMOS_POE, Q3 NMOS_POE, Q4 NMOS_POE, Q5 NMOS_POE, Q6 NMOS_POE, Q7 NMOS_POE, Q8 NMOS_POE, Q9 NMOS_POE, SW3 SW_Push, U1 LT4321, U14 DP83848C, U15 TMC429-I, U16 TMC2660C-PA, U2 LT4293, U3 STM32F407VETx, U4 NCP1117, U5 E48SC12010, X1 SXO53C, Y1 8MHz

Commit message: added programming pins
Parts:
- added C41: 1uF, Capacitor_SMD:C_0805_2012Metric_Pad1.15x1.40mm_HandSolder, F.Cu at (217.4, -68.4)
- added C42: 0.1uF, Capacitor_SMD:C_0805_2012Metric_Pad1.15x1.40mm_HandSolder, F.Cu at (222.1, -68.4)
- added REF**: MountingHole_3.2mm_M3, MountingHole:MountingHole_3.2mm_M3, F.Cu at (10.3, 16.0)
- added REF**: MountingHole_3.2mm_M3, MountingHole:MountingHole_3.2mm_M3, F.Cu at (99.2, 16.0)
- moved C10 236.6 mm to (77.9, 51.8), turned to 180 degrees
- moved C40 232.4 mm to (8.00, 60.2), turned to 270 degrees
- moved C4 215.1 mm to (57.5, 44.7)
- moved R32 208.2 mm to (87.0, 31.5)
- moved R20 202.3 mm to (89.0, -6.10)
- moved R35 201.7 mm to (86.5, 0.68)
- moved R36 199.5 mm to (85.0, 4.32)
- moved R31 199.3 mm to (87.2, 27.9)
- moved D4 198.7 mm to (178.4, -57.9)
- moved R30 197.9 mm to (87.8, 24.4)
- moved D5 192.9 mm to (179.0, -53.5)
- moved SW3 185.9 mm to (199.5, -60.5)
- moved C14 182.3 mm to (231.8, -42.7)
- moved C7 177.1 mm to (209.9, -44.7)
- moved Y1 175.5 mm to (214.8, -53.1)
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Connections:
- net Net-(U3-Pad72) renamed /SWDIO
- net Net-(U3-Pad76) renamed /SWCLK
- U3 pad 94: Net-(U3-Pad94) -> GND
Routing:
- net /Ethernet/RCLASS++: track 5.89 -> 55.4 mm
- net /Ethernet/RCLASS: track 2.54 -> 46.9 mm
- net GNDPWR: track 0.00 -> 30.1 mm, vias 0 -> 1
- net PWRGD: track 60.4 -> 87.0 mm
- net +3V3: track 0.00 -> 20.2 mm
- net Net-(RT5-Pad1): track 18.9 -> 5.95 mm
- net +12V: track 0.00 -> 11.1 mm
- net /Ethernet/VPORTP: track 53.0 -> 59.6 mm, vias 2 -> 4
- net Net-(RT8-Pad1): track 14.0 -> 20.4 mm
- net Net-(D1-Pad2): track 0.00 -> 5.72 mm, vias 0 -> 1
- net Net-(RT6-Pad1): track 16.3 -> 10.9 mm
- net Net-(D3-Pad2): track 0.00 -> 4.26 mm
- net VOUT-: track 9.50 -> 13.0 mm, vias 8 -> 9
- net Net-(RT7-Pad1): track 15.0 -> 16.8 mm
- added copper zone on B.Cu, net GND
- added copper zone on F.Cu, net GND
Other:
- outline, holes or cut-outs redrawn
- board text added: "<-PoE+ (30W)->"
- board text added: "<-PoE++(60W)->"

Commit message: burhhhhh sheeeeeeeeeeeeeeeeeesh
Parts:
- C24, C25, C26, C27, C28, C29, C30, C31, C32, C33, R21, R22, R33, R34: moved to B.Cu
- moved C11 243.7 mm to (48.8, 30.0), turned to 180 degrees
- moved C13 243.0 mm to (48.8, 32.1), turned to 180 degrees
- moved R21 235.0 mm to (61.3, 22.1), turned to 270 degrees
- moved R33 232.3 mm to (59.3, 22.1), turned to 270 degrees
- moved R34 230.7 mm to (65.7, 22.1), turned to 270 degrees
- moved R22 224.0 mm to (67.7, 22.1), turned to 270 degrees
- moved C24 217.2 mm to (69.7, 22.1), turned to 270 degrees
- moved C25 214.0 mm to (63.5, 22.1), turned to 270 degrees
- moved C29 211.3 mm to (80.5, 29.1), turned to 90 degrees
- moved C33 208.5 mm to (78.5, 33.6), turned to 90 degrees
- moved C12 136.5 mm to (184.5, -71.1)
- moved C6 134.3 mm to (185.3, -64.8)
- moved R37 119.4 mm to (171.1, -41.7)
- moved C2 102.1 mm to (216.0, 31.0)
- moved R2 94.7 mm to (218.6, -42.9)
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Connections:
- J1 pad 13: (no net) -> GNDPWR
Routing:
- net /Ethernet/TX+: track 0.00 -> 31.1 mm, vias 0 -> 3
- net /Ethernet/TX-: track 0.00 -> 28.8 mm, vias 0 -> 3
- net /Ethernet/RX-: track 0.00 -> 27.6 mm, vias 0 -> 1
- net /Ethernet/RX+: track 0.00 -> 26.7 mm, vias 0 -> 1
- net GND: track 0.00 -> 22.1 mm, vias 0 -> 7
- net Net-(C26-Pad1): track 0.00 -> 16.9 mm, vias 0 -> 3
- net +3V3: track 20.2 -> 33.3 mm, vias 0 -> 4
- net GNDPWR: track 30.1 -> 39.3 mm, vias 1 -> 2
- net Net-(U14-Pad34): track 0.00 -> 3.30 mm
- net Net-(R31-Pad1): track 0.00 -> 3.28 mm
- net Net-(R32-Pad1): track 0.00 -> 3.21 mm
- net Net-(R35-Pad1): track 0.00 -> 3.12 mm
- net CRS_DV: track 0.00 -> 2.89 mm
- net Net-(R30-Pad1): track 0.00 -> 2.54 mm
- net Net-(R20-Pad1): track 0.00 -> 2.03 mm
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- added copper zone on F.Cu, net +3V3
- removed copper zone on F.Cu, net GND

Commit message: Added motor control
Parts:
- moved U15 193.3 mm to (102.2, 41.8), turned to 180 degrees
- moved C17 175.9 mm to (123.3, 33.7)
- moved J2 175.5 mm to (122.0, 24.9)
- moved U16 160.3 mm to (123.9, 41.9)
- moved R24 149.1 mm to (106.8, 42.9), turned to -90 degrees
- moved R23 149.1 mm to (102.5, 47.0)
- moved R25 148.6 mm to (102.5, 37.9)
- moved C23 138.7 mm to (122.0, 50.2), turned to 180 degrees
- moved R26 138.6 mm to (115.8, 50.6)
- moved J3 129.9 mm to (99.5, 28.9)
- moved R27 127.6 mm to (118.0, 54.8)
- moved C14 127.3 mm to (129.9, 33.7)
- moved C15 126.1 mm to (122.0, 54.9)
- moved C19 117.6 mm to (112.1, 40.8), turned to 90 degrees
- moved R29 114.0 mm to (126.3, 55.2)
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Routing:
- net +12V: track 11.1 -> 76.5 mm, vias 0 -> 6
- net +3V3: track 33.3 -> 87.1 mm, vias 4 -> 8
- net Net-(J2-Pad2): track 0.00 -> 43.7 mm
- net Net-(J2-Pad4): track 0.00 -> 35.8 mm
- net GND: track 22.1 -> 52.5 mm, vias 7 -> 22
- net Net-(J3-Pad3): track 0.00 -> 24.1 mm
- net Net-(J3-Pad4): track 0.00 -> 23.4 mm, vias 0 -> 2
- net Net-(J2-Pad3): track 0.00 -> 23.1 mm
- net Net-(C18-Pad2): track 0.00 -> 22.0 mm, vias 0 -> 2
- net Net-(J2-Pad1): track 0.00 -> 21.6 mm
- net Net-(R26-Pad1): track 0.00 -> 17.4 mm, vias 0 -> 2
- net Net-(R28-Pad1): track 0.00 -> 15.8 mm, vias 0 -> 2
- net Net-(C16-Pad1): track 0.00 -> 10.2 mm
- net Net-(C15-Pad1): track 0.00 -> 8.76 mm
- net Net-(R25-Pad2): track 0.00 -> 7.03 mm
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- added copper zone on F.Cu, net GND
- added copper zone on F.Cu, net Net-(J2-Pad1)
- added copper zone on F.Cu, net Net-(J2-Pad2)
- added copper zone on F.Cu, net Net-(J2-Pad3)
- added copper zone on F.Cu, net Net-(J2-Pad4)
Other:
- net class Default removed

Commit message: Revert "Added motor control"
This reverts commit 7b2113a3a06210cf39fce9f6ba2f7b8593b46419.
Parts:
- moved U15 193.3 mm to (291.4, 81.3), turned to 0 degrees
- moved C17 175.9 mm to (290.7, 87.6)
- moved J2 175.5 mm to (290.4, 74.1)
- moved U16 160.3 mm to (279.9, 79.0)
- moved R24 149.1 mm to (255.1, 27.8), turned to 0 degrees
- moved R23 149.1 mm to (250.9, 33.7)
- moved R25 148.6 mm to (250.9, 30.7)
- moved C23 138.7 mm to (258.1, 23.6), turned to 0 degrees
- moved R26 138.6 mm to (251.9, 24.2)
- moved J3 129.9 mm to (229.3, 24.8)
- moved R27 127.6 mm to (244.4, 37.3)
- moved C14 127.3 mm to (231.8, -42.7)
- moved C15 126.1 mm to (246.2, 33.1)
- moved C19 117.6 mm to (229.5, 33.4), turned to 0 degrees
- moved R29 114.0 mm to (239.4, 40.6)
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Routing:
- net +12V: track 76.5 -> 11.1 mm, vias 6 -> 0
- net +3V3: track 87.1 -> 33.3 mm, vias 8 -> 4
- net Net-(J2-Pad2): track 43.7 -> 0.00 mm
- net Net-(J2-Pad4): track 35.8 -> 0.00 mm
- net GND: track 52.5 -> 22.1 mm, vias 22 -> 7
- net Net-(J3-Pad3): track 24.1 -> 0.00 mm
- net Net-(J3-Pad4): track 23.4 -> 0.00 mm, vias 2 -> 0
- net Net-(J2-Pad3): track 23.1 -> 0.00 mm
- net Net-(C18-Pad2): track 22.0 -> 0.00 mm, vias 2 -> 0
- net Net-(J2-Pad1): track 21.6 -> 0.00 mm
- net Net-(R26-Pad1): track 17.4 -> 0.00 mm, vias 2 -> 0
- net Net-(R28-Pad1): track 15.8 -> 0.00 mm, vias 2 -> 0
- net Net-(C16-Pad1): track 10.2 -> 0.00 mm
- net Net-(C15-Pad1): track 8.76 -> 0.00 mm
- net Net-(R25-Pad2): track 7.03 -> 0.00 mm
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- removed copper zone on F.Cu, net GND
- removed copper zone on F.Cu, net Net-(J2-Pad1)
- removed copper zone on F.Cu, net Net-(J2-Pad2)
- removed copper zone on F.Cu, net Net-(J2-Pad3)
- removed copper zone on F.Cu, net Net-(J2-Pad4)
Other:
- net class Default added: clearance 0.2, trace_width 0.25, via_dia 0.8, via_drill 0.4
